File: kicad/klorball35_left/klorball35_left.kicad_sch (KiCad schematic)
At the start: 0 parts

Commit message: Finishing footprints on left, starting schema
Parts:
- added SW1, SW10, SW11, SW12, SW13, SW14, SW15, SW16, SW17, SW18, SW2, SW3, SW4, SW5, SW6, SW7, SW8, SW9: SW_Push, keyswitches:Kailh_socket_PG1350_optional, symbol Library:SW_Push
- added U1: Helios, PCM_marbastlib-xp-promicroish:Helios_AC, symbol Library:Helios
Other:
- title: (none) -> Klorball35 Left
