File: kicad/klorball35_right/klorball35_right.kicad_sch (KiCad schematic)
At the start: 20 parts, among them J1 TRRS, SW1 SW_Push, SW10 SW_Push, SW11 SW_Push, SW12 SW_Push, SW13 SW_Push, SW14 SW_Push, SW15 SW_Push, SW16 SW_Push, SW17 SW_Push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

Commit message: Finishing left, start of right
Parts:
- removed SW10: SW_Push, keyswitches:Kailh_socket_PG1350_optional, symbol Switch:SW_Push
- added J2: Conn_01x07, Connector_PinHeader_2.54mm:PinHeader_1x07_P2.54mm_Vertical, symbol Connector_Generic:Conn_01x07
Connections:
- net +3V3: now also J2.6 (Pin_6)
- net GND: now also J2.7 (Pin_7)
- net INDEX_BOTTOM: now also U1.9 (P6); no longer U1.28 (P15)
- net INDEX_HOME: now also U1.28 (P15); no longer U1.11 (P8)
- net INDEX_THUMB: now also U1.2 (P1); no longer U1.21 (P22)
- net INDEX_TOP: now also U1.17 (P29); no longer U1.8 (P5)
- net INNER_BOTTOM: now also U1.10 (P7); no longer U1.27 (P14)
- net INNER_HOME: now also U1.29 (P16); no longer U1.10 (P7)
- net INNER_THUMB: now also U1.5 (P2); no longer U1.20 (P26)
- net INNER_TOP: now also U1.30 (P11); no longer U1.9 (P6)
- net MIDDLE_BOTTOM: now also U1.8 (P5); no longer U1.29 (P16)
- net MIDDLE_HOME: now also U1.27 (P14); no longer U1.12 (P9)
- net MIDDLE_TOP: now also U1.18 (P28); no longer U1.7 (P4)
- net PINKY_BOTTOM: now also U1.6 (P3); no longer U1.23 (P23)
- net PINKY_HOME: now also U1.25 (P12); no longer U1.26 (P13)
- net PINKY_TOP: now also U1.20 (P26); no longer U1.5 (P2)
- net RING_BOTTOM: now also U1.7 (P4); no longer U1.24 (P21)
- net RING_HOME: now also U1.26 (P13); no longer U1.25 (P12)
- net RING_TOP: now also U1.19 (P27); no longer U1.6 (P3)
- net MIDDLE_THUMB renamed MISO
- net MISO: now also J2.2 (Pin_2)
- net TRRS_RX: no longer names the net of J1.R1
- net TRRS_RX: no longer U1.2 (P1)
- new net CS: J2.1 (Pin_1), U1.24 (P21)
- new net MOSI: J2.3 (Pin_3), U1.23 (P23)
- new net SCK: J2.4 (Pin_4), U1.21 (P22)
Other:
- title: Klorball35 Left -> Klorball35 Right

Commit message: finishing right, start of gerbers
Connections:
- net INDEX_THUMB: now also U1.5 (P2); no longer U1.2 (P1)
- net INNER_THUMB: now also U1.2 (P1); no longer U1.5 (P2)
Changed lines of the file:
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@@
 		)
 	)
-	(label "INNER_THUMB"
+	(label "INDEX_THUMB"
 		(at 16.51 90.17 0)
 		(effects
@@
 		)
 	)
-	(label "INDEX_THUMB"
+	(label "INNER_THUMB"
 		(at 16.51 82.55 0)
 		(effects
