File: kicad/klorball35_right/klorball35_right.kicad_pcb (KiCad board)
At the start: 2 copper layers, 138.1 x 106.1 mm, 26 parts, among them J1 TRRS, J2 Conn_01x07, SW1 SW_Push, SW11 SW_Push, SW12 SW_Push, SW13 SW_Push, SW14 SW_Push, SW15 SW_Push, SW16 SW_Push, SW17 SW_Push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

Commit message: finishing right, start of gerbers
Connections:
- U1 pad 11: /INDEX_THUMB -> unconnected-(U1-P8-Pad11)
- U1 pad 12: /INNER_THUMB -> unconnected-(U1-P9-Pad12)_1
- U1 pad 2: unconnected-(U1-P1-Pad2)_1 -> /INNER_THUMB
- U1 pad 5: unconnected-(U1-P2-Pad5)_1 -> /INDEX_THUMB
Routing:
- net /PINKY_BOTTOM: track 12.5 -> 168.9 mm
- net /RING_BOTTOM: track 12.6 -> 145.9 mm
- net /MIDDLE_BOTTOM: track 12.7 -> 119.7 mm
- net /INDEX_THUMB: track 12.7 -> 119.4 mm
- net /INNER_THUMB: track 13.0 -> 108.0 mm
- net /INDEX_BOTTOM: track 12.7 -> 93.8 mm
- net /INNER_BOTTOM: track 12.7 -> 65.7 mm
- net /INNER_HOME: track 32.2 -> 30.6 mm
- net /INDEX_HOME: track 55.9 -> 54.5 mm
- net /RING_HOME: track 108.2 -> 106.9 mm
- net /PINKY_HOME: track 132.5 -> 131.6 mm

Commit message: Wrapping up, re-organizing.  Final gerbers and designs
Other:
- board text added: "KLORBALL35 Rev. 1.0"
Changed lines of the file:
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@@
 		(sheetname "/")
 		(sheetfile "klorball35_right.kicad_sch")
-		(attr through_hole)
+		(attr through_hole exclude_from_pos_files exclude_from_bom)
 		(fp_line
 			(start -7 7)
@@
 		(sheetname "/")
 		(sheetfile "klorball35_right.kicad_sch")
-		(attr through_hole)
+		(attr through_hole exclude_from_pos_files exclude_from_bom)
 		(fp_line
 			(start -7 -6)
@@
 		(sheetname "/")
 		(sheetfile "klorball35_right.kicad_sch")
-		(attr through_hole)
+		(attr through_hole exclude_from_pos_files exclude_from_bom)
 		(fp_line
 			(start -7 -6)
@@
 		(sheetname "/")
 		(sheetfile "klorball35_right.kicad_sch")
-		(attr through_hole)
+		(attr through_hole exclude_from_pos_files exclude_from_bom)
 		(fp_line
 			(start -7 7)
@@
 		(sheetname "/")
 		(sheetfile "klorball35_right.kicad_sch")
-		(attr through_hole)
+		(attr through_hole exclude_from_pos_files exclude_from_bom)
 		(fp_line
 			(start -7 7)
@@
 		(sheetname "/")
 		(sheetfile "klorball35_right.kicad_sch")
-		(attr through_hole)
+		(attr through_hole exclude_from_pos_files exclude_from_bom)
 		(fp_line
 			(start -7 -6.000001)
@@
 		(sheetname "/")
 		(sheetfile "klorball35_right.kicad_sch")
-		(attr through_hole)
+		(attr through_hole exclude_from_pos_files exclude_from_bom)
 		(fp_line
 			(start -7 7)
@@
 		(sheetname "/")
 		(sheetfile "klorball35_right.kicad_sch")
-		(attr through_hole)
+		(attr through_hole exclude_from_pos_files exclude_from_bom)
 		(fp_line
 			(start -7 7)
@@
 			(pinfunction "GND")
 			(pintype "power_in")
+			(zone_connect 2)
 		)
 		(pad "15" thru_hole circle
@@
 		(sheetname "/")
 		(sheetfile "klorball35_right.kicad_sch")
-		(attr through_hole)
+		(attr through_hole exclude_from_pos_files exclude_from_bom)
 		(fp_line
 			(start -7 -6)
@@
 		(sheetname "/")
 		(sheetfile "klorball35_right.kicad_sch")
-		(attr through_hole)
+		(attr through_hole exclude_from_pos_files exclude_from_bom)
 		(fp_line
 			(start -7 -5.999998)
@@
 		(sheetname "/")
 		(sheetfile "klorball35_right.kicad_sch")
-		(attr through_hole)
+		(attr through_hole exclude_from_pos_files exclude_from_bom)
 		(fp_line
 			(start 2.8 -2)
@@
 		(sheetname "/")
 		(sheetfile "klorball35_right.kicad_sch")
-		(attr through_hole)
+		(attr through_hole exclude_from_pos_files exclude_from_bom)
 		(fp_line
 			(start -7 7)
@@
 		(sheetname "/")
 		(sheetfile "klorball35_right.kicad_sch")
-		(attr through_hole)
+		(attr through_hole exclude_from_pos_files exclude_from_bom)
 		(fp_line
 			(start -7 -6)
@@
 		(sheetname "/")
 		(sheetfile "klorball35_right.kicad_sch")
-		(attr through_hole)
+		(attr through_hole exclude_from_pos_files exclude_from_bom)
 		(fp_line
 			(start -7 -6)
@@
 		(sheetname "/")
 		(sheetfile "klorball35_right.kicad_sch")
-		(attr through_hole)
+		(attr through_hole exclude_from_pos_files exclude_from_bom)
 		(fp_line
 			(start -7 7)
@@
 		(sheetname "/")
 		(sheetfile "klorball35_right.kicad_sch")
-		(attr through_hole)
+		(attr through_hole exclude_from_pos_files exclude_from_bom)
 		(fp_line
 			(start -1.38 16.619999)
@@
 		(sheetname "/")
 		(sheetfile "klorball35_right.kicad_sch")
-		(attr through_hole)
+		(attr through_hole exclude_from_pos_files exclude_from_bom)
 		(fp_line
 			(start -7 7)
@@
 		(sheetname "/")
 		(sheetfile "klorball35_right.kicad_sch")
-		(attr through_hole)
+		(attr through_hole exclude_from_pos_files exclude_from_bom)
 		(fp_line
 			(start -7 7)
@@
 		(sheetname "/")
 		(sheetfile "klorball35_right.kicad_sch")
-		(attr through_hole)
+		(attr through_hole exclude_from_pos_files exclude_from_bom)
 		(fp_line
 			(start -7 -6)
@@
 		(layer "Edge.Cuts")
 	)
+	(gr_text "KLORBALL35\nRev. 1.0"
+		(at 165.639549 157.339601 0)
+		(layer "F.SilkS")
+		(effects
+			(font
+				(size 1 1)
+				(thickness 0.2)
+				(bold yes)
+			)
+			(justify left bottom)
+		)
+	)
 	(segment
